Commit message: Make the panda URDFs portable via package:// mesh URIs
Both panda URDFs referenced meshes by absolute path on the machine the repo was
developed on (/home/tangles/Urop/ikflow/...), so loading the panda scene anywhere
else failed with a Drake "URI resolved to ... which does not exist" error. Point
every visual and collision mesh at
package://combining_kinematics/models/panda/collision_geometries/..., which
resolves through the package.xml that BuildEnv registers. All referenced meshes
are already vendored in that directory.

Co-Authored-By: Claude Opus 5 (1M context) <noreply@anthropic.com>
Claude-Session: https://claude.ai/code/session_01L4yYTpNhr43TZguTiSNH2B

File: models/panda/panda_no_hand.urdf (robot description, URDF)
Before this commit: robot panda, 9 links, 8 joints
Links:
- link panda_link0: geometry collision mesh filename=package://combining_kinematics/models/panda/collision_geome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; visual mesh filename=package://combining_kinematics/models/panda/collision_geome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
- link panda_link1: geometry collision mesh filename=package://combining_kinematics/models/panda/collision_geome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; visual mesh filename=package://combining_kinematics/models/panda/collision_geome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
- link panda_link2: geometry collision mesh filename=package://combining_kinematics/models/panda/collision_geome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; visual mesh filename=package://combining_kinematics/models/panda/collision_geome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
- link panda_link3: geometry collision mesh filename=package://combining_kinematics/models/panda/collision_geome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; visual mesh filename=package://combining_kinematics/models/panda/collision_geome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
- link panda_link4: geometry collision mesh filename=package://combining_kinematics/models/panda/collision_geome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; visual mesh filename=package://combining_kinematics/models/panda/collision_geome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
- link panda_link5: geometry collision mesh filename=package://combining_kinematics/models/panda/collision_geome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; visual mesh filename=package://combining_kinematics/models/panda/collision_geome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
- link panda_link6: geometry collision mesh filename=package://combining_kinematics/models/panda/collision_geome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; visual mesh filename=package://combining_kinematics/models/panda/collision_geome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
- link panda_link7: geometry collision mesh filename=package://combining_kinematics/models/panda/collision_geome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; visual mesh filename=package://combining_kinematics/models/panda/collision_geome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
